Commit message: add  2 new mjcf model + pipe to convert urdf to mjlab

File: models/bipedal_plateform/urdf/robot.urdf (robot description, URDF)
Before this commit: robot urdf, 18 links, 17 joints
Links:
- link torso_assembly: mass 1e-09 -> 5.3328; geometry collision mesh filename=package://assets/bearing_holder_upperbody.stl; collision mesh filename=package://assets/bearing_holder_upperbody.stl
Joints:
- joint anklex_left: origin xyz=8.43769e-15 -0.01594 0.02 rpy=1.5708 -1.56414 -1.84563e-13 -> xyz=8.77076e-15 -0.01594 0.02 rpy=1.5708 -1.56385 -1.68214e-13
- joint ankley_left: origin xyz=-2.77556e-16 -0.26 -0.02 rpy=-2.72876e-15 -1.04512e-15 -1.02684 -> xyz=-4.44089e-16 -0.26 -0.02 rpy=-1.88315e-15 -1.67074e-15 -0.955182
- joint ankley_right: origin xyz=-0.211522 -0.151191 0.02 rpy=3.14159 -6.73195e-15 1.16452 -> xyz=-0.221803 -0.135659 0.02 rpy=-3.14159 -6.73195e-15 1.16452
- joint hipx_left: origin xyz=-0.01897 0.0289 -0.09689 rpy=0.0663815 0.313138 2.36404 -> xyz=-0.01897 0.0289 -0.09689 rpy=0.0666815 0.313077 2.36501
- joint hipy_left: origin xyz=0.012638 0.0276823 -0.112055 rpy=1.64928 -0.538589 2.67351 -> xyz=0.012638 0.0276823 -0.112055 rpy=1.65228 -0.597222 2.66793
- joint hipy_right: origin xyz=0.012638 -0.0276823 -0.112055 rpy=-1.64778 0.505153 -2.75114 -> xyz=0.012638 -0.0276823 -0.112055 rpy=-1.64549 0.446566 -2.74613
- joint knee_left: origin xyz=-0.17 -0.294449 -0.0305 rpy=2.88538e-14 5.52989e-14 -1.39423 -> xyz=-0.17 -0.294449 -0.0305 rpy=2.3884e-15 -1.02851e-16 -1.52464
- joint knee_right: origin xyz=0.17 0.294449 -0.0305 rpy=3.14159 -1.64769e-13 -0.603194 -> xyz=0.17 0.294449 -0.0305 rpy=3.14159 -1.53592e-13 -0.544439

File: models/lerobot_humanoide/urdf/robot.urdf (robot description, URDF)
Before this commit: robot urdf, 27 links, 26 joints
Links:
- link forarm_subassembly: mass 1e-09 -> 0.119991
- link forarm_subassembly_2: mass 1e-09 -> 0.119991
- link shoulder1_subassembly: mass 1e-09 -> 0.0533612
- link shoulder1_subassembly_2: mass 1e-09 -> 0.0533612
- link shoulder2_subassembly: mass 1e-09 -> 0.813928; geometry collision mesh filename=package://assets/bearing_holder_upperbody.stl; collision mesh filename=package://assets/bearing_holder_upperbody.stl
- link shoulder2_subassembly_2: mass 1e-09 -> 0.813928; geometry collision mesh filename=package://assets/bearing_holder_upperbody.stl; collision mesh filename=package://assets/bearing_holder_upperbody.stl
- link shoulder3_subassembly: mass 1e-09 -> 0.356129; geometry collision mesh filename=package://assets/robstrideo0.stl; collision mesh filename=package://assets/shoulder3_part.stl
- link shoulder3_subassembly_2: mass 1e-09 -> 0.356129; geometry collision mesh filename=package://assets/robstrideo0.stl; collision mesh filename=package://assets/shoulder3_part.stl
- link torso_subassembly: mass 1.37476 -> 1.37455
- link torso_subassembly_2: mass 1e-09 -> 2.64598; geometry collision mesh filename=package://assets/bearing_holder_upperbody.stl; collision mesh filename=package://assets/bearing_holder_upperbody.stl
Joints:
- joint anklex_left: origin xyz=7.99361e-15 -0.01594 0.02 rpy=-1.5708 -1.51155 -3.14159 -> xyz=7.54952e-15 -0.01594 0.02 rpy=1.5708 -1.5708 0
- joint anklex_right: origin xyz=-5.55112e-15 -0.01594 0.02 rpy=1.5708 1.56918 -2.91336e-11 -> xyz=-6.32827e-15 -0.01594 0.02 rpy=1.5708 1.5708 0
- joint ankley_left: origin xyz=-3.88578e-16 -0.26 -0.02 rpy=-1.75167e-15 -2.14857e-15 -1.50866 -> xyz=-4.44089e-16 -0.26 -0.02 rpy=-1.55096e-15 -1.7069e-15 -0.955199
- joint ankley_right: origin xyz=-0.218697 -0.140611 0.02 rpy=3.14159 -6.83356e-15 1.16506 -> xyz=-0.222223 -0.134971 0.02 rpy=-3.14159 -6.92588e-15 1.16142
- joint hipx_left: origin xyz=-0.01897 0.0289 -0.09689 rpy=-0.00578336 0.31982 2.1331 -> xyz=-0.01897 0.0289 -0.09689 rpy=0.0593605 0.3145 2.3413
- joint hipx_right: origin xyz=-0.01897 -0.0289 -0.09689 rpy=-0.0611181 0.314174 -2.34698 -> xyz=-0.01897 -0.0289 -0.09689 rpy=-0.0593605 0.3145 -2.3413
- joint hipy_left: origin xyz=0.012638 0.0276823 -0.112055 rpy=1.72118 -1.1049 2.57926 -> xyz=0.012638 0.0276823 -0.112055 rpy=1.65232 -0.597994 2.66786
- joint hipy_right: origin xyz=0.012638 -0.0276823 -0.112055 rpy=-1.64283 0.361997 -2.73937 -> xyz=0.012638 -0.0276823 -0.112055 rpy=-1.64549 0.446566 -2.74613
- joint hipz_left: origin xyz=-0.00081771 0.13316 0.04164 rpy=-0.0308207 0.13784 1.32527 -> xyz=-0.000819037 0.13316 0.04164 rpy=-0.0475276 0.133035 1.20169
- joint hipz_right: origin xyz=-0.00081771 -0.133159 0.04164 rpy=0.0465927 0.133363 -1.20873 -> xyz=-0.000819037 -0.133159 0.04164 rpy=0.0475276 0.133035 -1.20169
- joint knee_left: origin xyz=-0.17 -0.294449 -0.0305 rpy=1.04567e-14 2.64358e-14 -1.47151 -> xyz=-0.17 -0.294449 -0.0305 rpy=3.0015e-14 6.08366e-14 -1.52464
- joint knee_right: origin xyz=0.17 0.294449 -0.0305 rpy=-3.14159 -1.47653e-14 -0.46045 -> xyz=0.17 0.294449 -0.0305 rpy=3.14159 -1.79424e-13 -0.547539
- joint left_hand_frame: origin xyz=0.23 2.77556e-17 0.027 rpy=-1.5708 3.26764e-16 -1.39521e-17 -> xyz=0.23 4.16334e-17 0.027 rpy=-1.5708 3.26764e-16 -1.39521e-17
- joint right_hand_frame: origin xyz=0.23 0 0.027 rpy=1.5708 1.67402e-18 1.01966e-15 -> xyz=0.23 5.55112e-17 0.027 rpy=1.5708 1.67402e-18 1.01966e-15
- joint upper_body: origin xyz=-0.0255415 4.03795e-07 0.036034 rpy=-3.14159 -3.99674e-17 6.83047e-18 -> xyz=-0.0255428 4.05842e-07 0.036034 rpy=-3.14159 -3.99674e-17 6.83047e-18
